File: clocks_pmod.kicad_sch (KiCad schematic)
At the start: 13 parts, among them J1 pmod, J2 25Mhz, J3 clk, U1 cjmcu-9833, U2 Si5351

Commit message: Add screeenshots
Other:
- company: (none) -> S59MZ
- title: (none) -> PMOD-CLOCKS
